Commit message: Updated version of the URDF file, should be fine now

File: hoap3.urdf (robot description, URDF)
Before this commit: robot hoap-3, 34 links, 33 joints
Joints:
- joint CHEST-L_SFE-joint: origin xyz=0.0 0.111 0.0 rpy=1.57079632679 -0.0 0.0 -> xyz=0.0 0.111 0.0 rpy=-1.57079632679 -0.0 0.0
- joint CHEST-R_SFE-joint: origin xyz=0.0 -0.111 0.0 rpy=1.57079632679 -0.0 0.0 -> xyz=0.0 -0.111 0.0 rpy=-1.57079632679 -0.0 0.0
- joint H_PAN-H_TILT-joint: origin xyz=0.015 0.0 0.103 rpy=1.57079632679 -0.0 0.0 -> xyz=0.015 0.0 0.103 rpy=-1.57079632679 -0.0 0.0
- joint L_AFE-L_AAA-joint: origin xyz=0.0 0.0 0.0 rpy=1.57079632679 -0.0 0.0 -> xyz=0.0 0.0 0.0 rpy=-1.57079632679 -0.0 0.0
- joint L_EB-L_WR-joint: origin xyz=0.0 0.133 0.0 rpy=1.57079632679 -0.0 0.0 -> xyz=0.0 0.133 0.0 rpy=-1.57079632679 -0.0 0.0
- joint L_LR-L_LAA-joint: origin xyz=0.0 0.0 0.0 rpy=0.0 -1.57079632679 0.0 -> xyz=0.0 0.0 0.0 rpy=1.57079632679 -1.57079632679 0.0
- joint L_SAA-L_SHR-joint: origin xyz=0.0 -0.111 0.0 rpy=0.0 -1.57079632679 0.0 -> xyz=0.0 -0.111 0.0 rpy=1.57079632679 -1.57079632679 0.0
- joint L_SFE-L_SAA-joint: origin xyz=0.0 0.0 0.0 rpy=0.0 -1.57079632679 0.0 -> xyz=0.0 0.0 0.0 rpy=1.57079632679 -1.57079632679 0.0
- joint R_AFE-R_AAA-joint: origin xyz=0.0 0.0 0.0 rpy=1.57079632679 -0.0 0.0 -> xyz=0.0 0.0 0.0 rpy=-1.57079632679 -0.0 0.0
- joint R_LR-R_LAA-joint: origin xyz=0.0 0.0 0.0 rpy=0.0 -1.57079632679 0.0 -> xyz=0.0 0.0 0.0 rpy=1.57079632679 -1.57079632679 0.0
- joint R_SAA-R_SHR-joint: origin xyz=0.0 -0.111 0.0 rpy=0.0 -1.57079632679 0.0 -> xyz=0.0 -0.111 0.0 rpy=1.57079632679 -1.57079632679 0.0
- joint R_SFE-R_SAA-joint: origin xyz=0.0 0.0 0.0 rpy=0.0 -1.57079632679 0.0 -> xyz=0.0 0.0 0.0 rpy=1.57079632679 -1.57079632679 0.0
- joint WAIST-L_LR-joint: origin xyz=-0.035 -0.055 -0.039 rpy=0.0 -1.57079632679 0.0 -> xyz=-0.035 -0.055 -0.039 rpy=-1.57079632679 1.57079632679 0.0
- joint WAIST-R_LR-joint: origin xyz=-0.035 -0.055 0.039 rpy=0.0 -1.57079632679 0.0 -> xyz=-0.035 -0.055 0.039 rpy=-1.57079632679 1.57079632679 0.0

Commit message: Split HOAP3 hands in wrist and hand.
While here:
- Base -> base_link
- *-*-joint -> *_*_joint

File: hoap3.urdf (robot description, URDF)
Before this commit: robot hoap-3, 34 links, 33 joints
Links:
- removed link Base
- added link L_HAND; visual mesh filename=package://hoap3_description/meshes/LHAND.dae
- added link R_HAND; visual mesh filename=package://hoap3_description/meshes/RHAND.dae
- added link base_link
Joints:
- removed joint Base-CHEST-joint
- removed joint CHEST-H_PAN-joint
- removed joint CHEST-L_SFE-joint
- removed joint CHEST-R_SFE-joint
- removed joint CHEST-WAIST-joint
- removed joint H_PAN-H_TILT-joint
- removed joint H_ROLL-EYE-joint
- removed joint H_ROLL-HEAD-joint
- removed joint H_ROLL-LEYE-joint
- removed joint H_ROLL-REYE-joint
- removed joint H_TILT-H_ROLL-joint
- removed joint L_AAA-L_FOOT-joint
- removed joint L_AFE-L_AAA-joint
- removed joint L_EB-L_WR-joint
- removed joint L_KN-L_AFE-joint
- removed joint L_LAA-L_LFE-joint
- removed joint L_LFE-L_KN-joint
- removed joint L_LR-L_LAA-joint
- removed joint L_SAA-L_SHR-joint
- removed joint L_SFE-L_SAA-joint
- removed joint L_SHR-L_EB-joint
- removed joint R_AAA-R_FOOT-joint
- removed joint R_AFE-R_AAA-joint
- removed joint R_EB-R_WR-joint
- removed joint R_KN-R_AFE-joint
- removed joint R_LAA-R_LFE-joint
- removed joint R_LFE-R_KN-joint
- removed joint R_LR-R_LAA-joint
- removed joint R_SAA-R_SHR-joint
- removed joint R_SFE-R_SAA-joint
- removed joint R_SHR-R_EB-joint
- removed joint WAIST-L_LR-joint
- removed joint WAIST-R_LR-joint
- added joint Base_CHEST_joint: type fixed, parent base_link, child CHEST, origin xyz=0.0 0.0 0.5 rpy=0.0 -0.0 0.0
- added joint CHEST_H_PAN_joint: type revolute, parent CHEST, child H_PAN, origin xyz=0.0 0.0 0.0 rpy=0.0 -0.0 0.0, axis 0 0 1, limit lower=-1.0471975512 upper=1.0471975512 effort=100 velocity=100
- added joint CHEST_L_SFE_joint: type revolute, parent CHEST, child L_SFE, origin xyz=0.0 0.111 0.0 rpy=-1.57079632679 -0.0 0.0, axis 0 0 1, limit lower=-1.57079632679 upper=2.44346095279 effort=100 velocity=100
- added joint CHEST_R_SFE_joint: type revolute, parent CHEST, child R_SFE, origin xyz=0.0 -0.111 0.0 rpy=-1.57079632679 -0.0 0.0, axis 0 0 1, limit lower=-1.57079632679 upper=2.44346095279 effort=100 velocity=100
- added joint CHEST_WAIST_joint: type revolute, parent CHEST, child WAIST, origin xyz=0.035 0.0 -0.125 rpy=1.57079632679 -0.0 0.0, axis 0 0 1, limit lower=0.0 upper=0.610865238198 effort=100 velocity=100
- added joint H_PAN_H_TILT_joint: type revolute, parent H_PAN, child H_TILT, origin xyz=0.015 0.0 0.103 rpy=-1.57079632679 -0.0 0.0, axis 0 0 -1, limit lower=-0.785398163397 upper=0.261799387799 effort=100 velocity=100
- added joint H_ROLL_EYE_joint: type fixed, parent H_ROLL, child EYE, origin xyz=0.06 0.004 0.0 rpy=0.0 -0.0 0.0
- added joint H_ROLL_HEAD_joint: type fixed, parent H_ROLL, child HEAD, origin xyz=0.0 -0.07 0.0 rpy=0.0 -0.0 0.0
- added joint H_ROLL_LEYE_joint: type fixed, parent H_ROLL, child LEYE, origin xyz=0.05 0.004 0.03 rpy=0.0 -0.0 0.0
- added joint H_ROLL_REYE_joint: type fixed, parent H_ROLL, child REYE, origin xyz=0.05 0.004 -0.03 rpy=0.0 -0.0 0.0
- added joint H_TILT_H_ROLL_joint: type revolute, parent H_TILT, child H_ROLL, origin xyz=0.0 0.0 0.0 rpy=0.0 -0.0 0.0, axis -1 0 0, limit lower=-0.261799387799 upper=0.261799387799 effort=100 velocity=100
- added joint L_AAA_L_FOOT_joint: type fixed, parent L_AAA, child L_FOOT, origin xyz=-0.04 -0.005 0.014 rpy=0.0 -0.0 0.0
- added joint L_AFE_L_AAA_joint: type revolute, parent L_AFE, child L_AAA, origin xyz=0.0 0.0 0.0 rpy=-1.57079632679 -0.0 0.0, axis 0 0 1, limit lower=-0.436332312999 upper=0.436332312999 effort=100 velocity=100
- added joint L_EB_L_WR_joint: type revolute, parent L_EB, child L_WR, origin xyz=0.0 0.0478 0.0 rpy=-1.57079632679 -0.0 0.0, axis 0 0 1, limit lower=-1.57079632679 upper=1.57079632679 effort=100 velocity=100
- added joint L_KN_L_AFE_joint: type revolute, parent L_KN, child L_AFE, origin xyz=-0.105 0.0 0.0 rpy=0.0 -0.0 0.0, axis 0 0 1, limit lower=-1.0471975512 upper=1.0471975512 effort=100 velocity=100
- added joint L_LAA_L_LFE_joint: type revolute, parent L_LAA, child L_LFE, origin xyz=0.0 0.0 0.0 rpy=1.57079632679 -0.0 0.0, axis 0 0 1, limit lower=-1.3962634016 upper=1.2217304764 effort=100 velocity=100
- added joint L_LFE_L_KN_joint: type revolute, parent L_LFE, child L_KN, origin xyz=-0.105 0.0 0.0 rpy=0.0 -0.0 0.0, axis 0 0 1, limit lower=0.0872664625997 upper=2.26892802759 effort=100 velocity=100
- added joint L_LR_L_LAA_joint: type revolute, parent L_LR, child L_LAA, origin xyz=0.0 0.0 0.0 rpy=1.57079632679 -1.57079632679 0.0, axis 0 0 1, limit lower=-0.349065850399 upper=0.523598775598 effort=100 velocity=100
- added joint L_SAA_L_SHR_joint: type revolute, parent L_SAA, child L_SHR, origin xyz=0.0 -0.111 0.0 rpy=1.57079632679 -1.57079632679 0.0, axis 0 0 1, limit lower=-1.58824961931 upper=1.58824961931 effort=100 velocity=100
- added joint L_SFE_L_SAA_joint: type revolute, parent L_SFE, child L_SAA, origin xyz=0.0 0.0 0.0 rpy=1.57079632679 -1.57079632679 0.0, axis 0 0 1, limit lower=0.0 upper=1.57079632679 effort=100 velocity=100
- added joint L_SHR_L_EB_joint: type revolute, parent L_SHR, child L_EB, origin xyz=0.0 0.0 0.0 rpy=1.57079632679 -0.0 0.0, axis 0 0 1, limit lower=-2.00712863979 upper=0.0 effort=100 velocity=100
- added joint L_WR_L_HAND_joint: type fixed, parent L_WR, child L_HAND, origin xyz=0.0 0.0 0.055 rpy=0.0 0.0 0.0
- added joint R_AAA_R_FOOT_joint: type fixed, parent R_AAA, child R_FOOT, origin xyz=-0.04 0.005 0.014 rpy=0.0 -0.0 0.0
- added joint R_AFE_R_AAA_joint: type revolute, parent R_AFE, child R_AAA, origin xyz=0.0 0.0 0.0 rpy=-1.57079632679 -0.0 0.0, axis 0 0 1, limit lower=-0.436332312999 upper=0.436332312999 effort=100 velocity=100
- added joint R_EB_R_WR_joint: type revolute, parent R_EB, child R_WR, origin xyz=0.0 0.0478 0.0 rpy=1.57079632679 -0.0 0.0, axis 0 0 1, limit lower=-1.0471975512 upper=1.0471975512 effort=100 velocity=100
- added joint R_KN_R_AFE_joint: type revolute, parent R_KN, child R_AFE, origin xyz=-0.105 0.0 0.0 rpy=0.0 -0.0 0.0, axis 0 0 1, limit lower=-1.0471975512 upper=1.0471975512 effort=100 velocity=100
- added joint R_LAA_R_LFE_joint: type revolute, parent R_LAA, child R_LFE, origin xyz=0.0 0.0 0.0 rpy=1.57079632679 -0.0 0.0, axis 0 0 1, limit lower=-1.3962634016 upper=1.2217304764 effort=100 velocity=100
- added joint R_LFE_R_KN_joint: type revolute, parent R_LFE, child R_KN, origin xyz=-0.105 0.0 0.0 rpy=0.0 -0.0 0.0, axis 0 0 1, limit lower=0.0872664625997 upper=2.26892802759 effort=100 velocity=100
- added joint R_LR_R_LAA_joint: type revolute, parent R_LR, child R_LAA, origin xyz=0.0 0.0 0.0 rpy=1.57079632679 -1.57079632679 0.0, axis 0 0 1, limit lower=-0.523598775598 upper=0.349065850399 effort=100 velocity=100
- added joint R_SAA_R_SHR_joint: type revolute, parent R_SAA, child R_SHR, origin xyz=0.0 -0.111 0.0 rpy=1.57079632679 -1.57079632679 0.0, axis 0 0 1, limit lower=-1.57079632679 upper=1.57079632679 effort=100 velocity=100
- added joint R_SFE_R_SAA_joint: type revolute, parent R_SFE, child R_SAA, origin xyz=0.0 0.0 0.0 rpy=1.57079632679 -1.57079632679 0.0, axis 0 0 1, limit lower=-1.57079632679 upper=0.0 effort=100 velocity=100
- added joint R_SHR_R_EB_joint: type revolute, parent R_SHR, child R_EB, origin xyz=0.0 0.0 0.0 rpy=1.57079632679 -0.0 0.0, axis 0 0 1, limit lower=-2.00712863979 upper=0.0 effort=100 velocity=100
- added joint R_WR_R_HAND_joint: type fixed, parent R_WR, child R_HAND, origin xyz=0.0 0.0 -0.055 rpy=0.0 0.0 0.0
- added joint WAIST_L_LR_joint: type revolute, parent WAIST, child L_LR, origin xyz=-0.035 -0.055 -0.039 rpy=-1.57079632679 1.57079632679 0.0, axis 0 0 1, limit lower=-0.523598775598 upper=1.57079632679 effort=100 velocity=100
- added joint WAIST_R_LR_joint: type revolute, parent WAIST, child R_LR, origin xyz=-0.035 -0.055 0.039 rpy=-1.57079632679 1.57079632679 0.0, axis 0 0 1, limit lower=-1.57079632679 upper=0.523598775598 effort=100 velocity=100

Commit message: Set WAIST as the fixed link

File: hoap3.urdf (robot description, URDF)
Before this commit: robot hoap3, 36 links, 35 joints
Joints:
- removed joint Base_CHEST_joint
- removed joint CHEST_WAIST_joint
- added joint WAIST_CHEST_joint: type revolute, parent WAIST, child CHEST, origin xyz=-0.0 0.0 0.0 rpy=-1.57079632679 -0.0 0.0, axis 0 1 0, limit lower=0.0 upper=0.610865238198 effort=100 velocity=100
- added joint base_link_WAIST_joint: type fixed, parent base_link, child WAIST, origin xyz=0.0 0.0 0.0 rpy=1.57079632679 -0.0 0.0
- joint CHEST_H_PAN_joint: origin xyz=0.0 0.0 0.0 rpy=0.0 -0.0 0.0 -> xyz=-0.035 0.0 0.125 rpy=0.0 -0.0 0.0
- joint CHEST_L_SFE_joint: origin xyz=0.0 0.111 0.0 rpy=-1.57079632679 -0.0 0.0 -> xyz=-0.035 0.111 0.125 rpy=-1.57079632679 -0.0 0.0
- joint CHEST_R_SFE_joint: origin xyz=0.0 -0.111 0.0 rpy=-1.57079632679 -0.0 0.0 -> xyz=-0.035 -0.111 0.125 rpy=-1.57079632679 -0.0 0.0
